Commit message: fix scale in stl and edit urdf

File: src/kirin/urdf/kirin.urdf (robot description, URDF)
Before this commit: robot kirin, 2 links, 1 joints
Links:
- added link theta_link; visual mesh filename=package://kirin/resources/theta.stl
- link fix_base: geometry visual mesh filename=package://kirin/resources/fix.stl
Joints:
- added joint theta_joint: type fixed, parent fix_base, child theta_link, origin xyz=0.0 0.0 0.5 rpy=0.0 0.0 0.0
- joint base_joint: origin (none) -> xyz=0.0 0.0 0.0 rpy=0.0 0.0 0.0

Commit message: modify urdf to display in approximate correct position

File: src/kirin/urdf/kirin.urdf (robot description, URDF)
Before this commit: robot kirin, 3 links, 2 joints
Links:
- added link phi_extend_link; visual mesh filename=package://kirin/resources/light/phi_extend.stl
- added link phi_link; visual mesh filename=package://kirin/resources/light/phi.stl
- added link r_link; visual mesh filename=package://kirin/resources/light/r.stl
- added link z_link; visual mesh filename=package://kirin/resources/light/z.stl
- link fix_base: geometry visual mesh filename=package://kirin/resources/light/fix.stl
- link theta_link: geometry visual mesh filename=package://kirin/resources/light/theta.stl
Joints:
- added joint phi_extend_joint: type fixed, parent r_link, child phi_extend_link, origin xyz=0.4 0.0 -0.2 rpy=0.0 0.0 0.0
- added joint phi_joint: type fixed, parent r_link, child phi_link, origin xyz=0.4 0.0 -0.1 rpy=0.0 0.0 0.0
- added joint r_joint: type fixed, parent z_link, child r_link, origin xyz=0.5 0.0 -0.2 rpy=0.0 0.0 0.0
- added joint z_joint: type fixed, parent theta_link, child z_link, origin xyz=0.0 0.0 0.7 rpy=0.0 0.0 0.0
- joint theta_joint: origin xyz=0.0 0.0 0.5 rpy=0.0 0.0 0.0 -> xyz=0.0 0.0 0.1 rpy=0.0 0.0 0.0

Commit message: modify joint type

File: src/kirin/urdf/kirin.urdf (robot description, URDF)
Before this commit: robot kirin, 7 links, 6 joints
Joints:
- joint phi_extend_joint: axis (none) -> 0.0 0.0 1.0; limit (none) -> lower=-3.14 upper=3.14 effort=10.0 velocity=31.4; type fixed -> revolute
- joint phi_joint: axis (none) -> 0.0 0.0 1.0; limit (none) -> lower=-3.14 upper=3.14 effort=10.0 velocity=31.4; type fixed -> revolute
- joint r_joint: axis (none) -> 1.0 0.0 0.0; limit (none) -> lower=0.0 upper=0.8 effort=100 velocity=5.0; origin xyz=0.5 0.0 -0.2 rpy=0.0 0.0 0.0 -> xyz=0.1 0.0 -0.1 rpy=0.0 0.0 0.0; type fixed -> prismatic
- joint theta_joint: axis (none) -> 0.0 0.0 1.0; type fixed -> continuous
- joint z_joint: axis (none) -> 0.0 0.0 1.0; limit (none) -> lower=0.1 upper=0.6 effort=100 velocity=2.0; origin xyz=0.0 0.0 0.7 rpy=0.0 0.0 0.0 -> xyz=0.0 0.0 0.3 rpy=0.0 0.0 0.0; type fixed -> prismatic

Commit message: modified detail parameter in urdf

File: src/kirin/urdf/kirin.urdf (robot description, URDF)
Before this commit: robot kirin, 7 links, 6 joints
Links:
- added link jagariko; visual mesh filename=package://kirin/resources/jagariko.stl
- added link jagariko_top
Joints:
- added joint jagariko_joint: type fixed, parent base_link, child jagariko, origin xyz=0.8 0.2 0.0 rpy=0.0 0.0 1.57
- added joint jagariko_top_joint: type fixed, parent jagariko, child jagariko_top, origin xyz=0.0 0.0 0.08 rpy=0.0 0.0 0.0
- joint phi_extend_joint: origin xyz=0.4 0.0 -0.2 rpy=0.0 0.0 0.0 -> xyz=0.345 0.0 -0.0235 rpy=0.0 0.0 0.0
- joint phi_joint: origin xyz=0.4 0.0 -0.1 rpy=0.0 0.0 0.0 -> xyz=0.345 0.0 -0.0235 rpy=0.0 0.0 0.0
- joint r_joint: limit lower=0.0 upper=0.8 effort=100 velocity=5.0 -> lower=0.0 upper=0.413 effort=100 velocity=5.0; origin xyz=0.1 0.0 -0.1 rpy=0.0 0.0 0.0 -> xyz=0.201 0.0 0.0 rpy=0.0 0.0 0.0
- joint theta_joint: origin xyz=0.0 0.0 0.1 rpy=0.0 0.0 0.0 -> xyz=0.0 0.0 0.022 rpy=0.0 0.0 0.0
- joint z_joint: limit lower=0.1 upper=0.6 effort=100 velocity=2.0 -> lower=0.0 upper=0.15 effort=100 velocity=2.0; origin xyz=0.0 0.0 0.3 rpy=0.0 0.0 0.0 -> xyz=0.0 0.0 0.128 rpy=0.0 0.0 0.0
