Commit message: add field stl file and move file position

File: src/kirin/urdf/field.urdf.xacro (robot description, xacro)
@@ -4,5 +4,5 @@
       <origin xyz="0.0 0.0 0.0" rpy="0.0 0.0 3.14159265"/>
       <geometry>
-        <mesh filename="package://kirin/resources/light_field.dae"/>
+        <mesh filename="package://kirin/resources/light/field.dae"/>
       </geometry>
     </visual>
