Commit message: change from urdf to xacro

File: src/kirin/urdf/kirin.urdf.xacro (robot description, xacro)
@@ -1,97 +1,61 @@
 <robot name="kirin">
-  <link name="base_link"/>
+  <material name="default">
+    <color rgba="0.7 0.7 0.7 1.0"/>
+  </material>
+  <!-- link settings -->
   <link name="fix_base">
     <visual name="">
-      <origin xyz="0.0 0.0 0.0" rpy="0.0 0.0 -1.57"/>
+      <origin xyz="0.0 0.0 0.0" rpy="0.0 0.0 ${-pi/2}"/>
       <geometry>
         <mesh filename="package://kirin/resources/light/fix.stl"/>
       </geometry>
-      <material name="">
-        <color rgba="0.7 0.7 0.7 1.0"/>
-      </material>
+      <material name="default"/>
     </visual>
   </link>
   <link name="theta_link">
     <visual name="">
-      <origin xyz="0.0 0.0 0.0" rpy="0.0 0.0 1.57"/>
+      <origin xyz="0.0 0.0 0.0" rpy="0.0 0.0 ${pi/2}"/>
       <geometry>
         <mesh filename="package://kirin/resources/light/theta.stl"/>
       </geometry>
-      <material name="">
-        <color rgba="0.7 0.7 0.7 1.0"/>
-      </material>
+      <material name="default"/>
     </visual>
   </link>
   <link name="z_link">
     <visual name="">
-      <origin xyz="0.0 0.0 0.0" rpy="0.0 0.0 1.57"/>
+      <origin xyz="0.0 0.0 0.0" rpy="0.0 0.0 ${pi/2}"/>
       <geometry>
         <mesh filename="package://kirin/resources/light/z.stl"/>
       </geometry>
-      <material name="">
-        <color rgba="0.7 0.7 0.7 1.0"/>
-      </material>
+      <material name="default"/>
     </visual>
   </link>
   <link name="r_link">
     <visual name="">
-      <origin xyz="0.1725 0.0 0.0" rpy="0.0 0.0 1.57"/>
+      <origin xyz="0.1725 0.0 0.0" rpy="0.0 0.0 ${pi/2}"/>
       <geometry>
         <mesh filename="package://kirin/resources/light/r.stl"/>
       </geometry>
-      <material name="">
-        <color rgba="0.7 0.7 0.7 1.0"/>
-      </material>
+      <material name="default"/>
     </visual>
   </link>
   <link name="phi_link">
     <visual name="">
-      <origin xyz="0.0 0.0 0.0" rpy="0.0 0.0 1.57"/>
+      <origin xyz="0.0 0.0 0.0" rpy="0.0 0.0 ${pi/2}"/>
       <geometry>
         <mesh filename="package://kirin/resources/light/phi.stl"/>
       </geometry>
-      <material name="">
-        <color rgba="0.7 0.7 0.7 1.0"/>
-      </material>
+      <material name="default"/>
     </visual>
   </link>
   <link name="phi_extend_link">
     <visual name="">
-      <origin xyz="0.0 0.0 0.0" rpy="0.0 0.0 1.57"/>
+      <origin xyz="0.0 0.0 0.0" rpy="0.0 0.0 ${pi/2}"/>
       <geometry>
         <mesh filename="package://kirin/resources/light/phi_extend.stl"/>
       </geometry>
-      <material name="">
-        <color rgba="0.7 0.7 0.7 1.0"/>
-      </material>
+      <material name="default"/>
     </visual>
   </link>
-  <link name="jagariko">
-    <visual name="">
-      <origin xyz="0.0 0.0 0.0" rpy="0.0 0.0 1.57"/>
-      <geometry>
-        <mesh filename="package://kirin/resources/jagariko.stl"/>
-      </geometry>
-      <material name="">
-        <color rgba="0.7 0.7 0.7 1.0"/>
-      </material>
-    </visual>
-  </link>
-  <link name="jagariko_top"/>
-  <joint name="base_joint" type="fixed">
-    <parent link="base_link"/>
-    <child link="fix_base"/>
-    <origin xyz="0.0 0.0 0.0" rpy="0.0 0.0 0.0"/>
-  </joint>
-  <joint name="jagariko_joint" type="fixed">
-    <parent link="base_link"/>
-    <child link="jagariko"/>
-    <origin xyz="0.8 0.2 0.0" rpy="0.0 0.0 1.57"/>
-  </joint>
-  <joint name="jagariko_top_joint" type="fixed">
-    <parent link="jagariko"/>
-    <child link="jagariko_top"/>
-    <origin xyz="0.0 0.0 0.08" rpy="0.0 0.0 0.0"/>
-  </joint>
   <joint name="theta_joint" type="continuous">
     <parent link="fix_base"/>
@@ -119,5 +83,5 @@
     <origin xyz="0.345 0.0 -0.0235" rpy="0.0 0.0 0.0"/>
     <axis xyz="0.0 0.0 1.0"/>
-    <limit lower="-3.14" upper="3.14" effort="10.0" velocity="31.4"/>
+    <limit lower="${-pi}" upper="${pi}" effort="10.0" velocity="${10*pi}"/>
   </joint>
   <joint name="phi_extend_joint" type="revolute">
@@ -126,5 +90,5 @@
     <origin xyz="0.345 0.0 -0.0235" rpy="0.0 0.0 0.0"/>
     <axis xyz="0.0 0.0 1.0"/>
-    <limit lower="-3.14" upper="3.14" effort="10.0" velocity="31.4"/>
+    <limit lower="${-pi}" upper="${pi}" effort="10.0" velocity="${10*pi}"/>
   </joint>
 </robot>

Commit message: fix fix_base angle

File: src/kirin/urdf/kirin.urdf.xacro (robot description, xacro)
@@ -6,5 +6,5 @@
   <link name="fix_base">
     <visual name="">
-      <origin xyz="0.0 0.0 0.0" rpy="0.0 0.0 ${-pi/2}"/>
+      <origin xyz="0.0 0.0 0.0" rpy="0.0 0.0 ${pi/2}"/>
       <geometry>
         <mesh filename="package://kirin/resources/light/fix.stl"/>

Commit message: world coord manual moved properly

File: src/kirin/urdf/kirin.urdf.xacro (robot description, xacro)
@@ -1,3 +1,3 @@
-<robot name="kirin">
+<robot name="kirin" xmlns:xacro="http://ros.org/wiki/xacro">
   <material name="default">
     <color rgba="0.7 0.7 0.7 1.0"/>
@@ -49,4 +49,7 @@
     </visual>
   </link>
+  <link name="top_bellows"/>
+  <link name="left_bellows"/>
+  <link name="right_bellows"/>
   <link name="phi_extend_link">
     <visual name="">
@@ -86,4 +89,21 @@
     <limit lower="${-pi}" upper="${pi}" effort="10.0" velocity="${10*pi}"/>
   </joint>
+  <xacro:property name="bellows_d" value="0.1"/>
+  <xacro:property name="bellows_z" value="-0.042"/>
+  <joint name="top_bellows_joint" type="fixed">
+    <parent link="phi_link"/>
+    <child link="top_bellows"/>
+    <origin xyz="0.05 0.0 ${bellows_z}" rpy="0.0 0.0 0.0"/>
+  </joint>
+  <joint name="left_bellows_joint" type="fixed">
+    <parent link="top_bellows"/>
+    <child link="left_bellows"/>
+    <origin xyz="-${bellows_d} -${bellows_d} 0.0" rpy="0.0 0.0 0.0"/>
+  </joint>
+  <joint name="right_bellows_joint" type="fixed">
+    <parent link="top_bellows"/>
+    <child link="right_bellows"/>
+    <origin xyz="-${bellows_d} ${bellows_d} 0.0" rpy="0.0 0.0 0.0"/>
+  </joint>
   <joint name="phi_extend_joint" type="revolute">
     <parent link="r_link"/>

Commit message: add hand tool manager

File: src/kirin/urdf/kirin.urdf.xacro (robot description, xacro)
@@ -40,7 +40,8 @@
     </visual>
   </link>
-  <link name="phi_link">
+  <link name="phi_link_base"/>
+  <!-- <link name="phi_link">
     <visual name="">
-      <origin xyz="0.0 0.0 0.0" rpy="0.0 0.0 ${pi/2}"/>
+      <origin xyz="0.0 0.0 0.0" rpy="0.0 0.0 0.0"/>
       <geometry>
         <mesh filename="package://kirin/resources/light/phi.stl"/>
@@ -54,5 +55,5 @@
   <link name="phi_extend_link">
     <visual name="">
-      <origin xyz="0.0 0.0 0.0" rpy="0.0 0.0 ${pi/2}"/>
+      <origin xyz="0.0 0.0 0.0" rpy="0.0 0.0 0.0"/>
       <geometry>
         <mesh filename="package://kirin/resources/light/phi_extend.stl"/>
@@ -60,5 +61,5 @@
       <material name="default"/>
     </visual>
-  </link>
+  </link> -->
   <!-- joint settings -->
   <joint name="theta_joint" type="continuous">
@@ -84,10 +85,10 @@
   <joint name="phi_joint" type="revolute">
     <parent link="r_link"/>
-    <child link="phi_link"/>
+    <child link="phi_link_base"/>
     <origin xyz="0.345 0.0 -0.0235" rpy="0.0 0.0 0.0"/>
     <axis xyz="0.0 0.0 1.0"/>
     <limit lower="${-pi}" upper="${pi}" effort="10.0" velocity="${10*pi}"/>
   </joint>
-  <xacro:property name="bellows_d" value="0.1"/>
+  <!-- <xacro:property name="bellows_d" value="0.1"/>
   <xacro:property name="bellows_z" value="-0.042"/>
   <joint name="top_bellows_joint" type="fixed">
@@ -112,4 +113,4 @@
     <axis xyz="0.0 0.0 1.0"/>
     <limit lower="${-pi}" upper="${pi}" effort="10.0" velocity="${10*pi}"/>
-  </joint>
+  </joint> -->
 </robot>

Commit message: broadcast bellows frame in tool manager

File: src/kirin/urdf/kirin.urdf.xacro (robot description, xacro)
@@ -40,26 +40,5 @@
     </visual>
   </link>
-  <link name="phi_link_base"/>
-  <!-- <link name="phi_link">
-    <visual name="">
-      <origin xyz="0.0 0.0 0.0" rpy="0.0 0.0 0.0"/>
-      <geometry>
-        <mesh filename="package://kirin/resources/light/phi.stl"/>
-      </geometry>
-      <material name="default"/>
-    </visual>
-  </link>
-  <link name="top_bellows"/>
-  <link name="left_bellows"/>
-  <link name="right_bellows"/>
-  <link name="phi_extend_link">
-    <visual name="">
-      <origin xyz="0.0 0.0 0.0" rpy="0.0 0.0 0.0"/>
-      <geometry>
-        <mesh filename="package://kirin/resources/light/phi_extend.stl"/>
-      </geometry>
-      <material name="default"/>
-    </visual>
-  </link> -->
+  <link name="phi_link"/>
   <!-- joint settings -->
   <joint name="theta_joint" type="continuous">
@@ -85,32 +64,8 @@
   <joint name="phi_joint" type="revolute">
     <parent link="r_link"/>
-    <child link="phi_link_base"/>
+    <child link="phi_link"/>
     <origin xyz="0.345 0.0 -0.0235" rpy="0.0 0.0 0.0"/>
     <axis xyz="0.0 0.0 1.0"/>
     <limit lower="${-pi}" upper="${pi}" effort="10.0" velocity="${10*pi}"/>
   </joint>
-  <!-- <xacro:property name="bellows_d" value="0.1"/>
-  <xacro:property name="bellows_z" value="-0.042"/>
-  <joint name="top_bellows_joint" type="fixed">
-    <parent link="phi_link"/>
-    <child link="top_bellows"/>
-    <origin xyz="0.05 0.0 ${bellows_z}" rpy="0.0 0.0 0.0"/>
-  </joint>
-  <joint name="left_bellows_joint" type="fixed">
-    <parent link="top_bellows"/>
-    <child link="left_bellows"/>
-    <origin xyz="-${bellows_d} -${bellows_d} 0.0" rpy="0.0 0.0 0.0"/>
-  </joint>
-  <joint name="right_bellows_joint" type="fixed">
-    <parent link="top_bellows"/>
-    <child link="right_bellows"/>
-    <origin xyz="-${bellows_d} ${bellows_d} 0.0" rpy="0.0 0.0 0.0"/>
-  </joint>
-  <joint name="phi_extend_joint" type="revolute">
-    <parent link="r_link"/>
-    <child link="phi_extend_link"/>
-    <origin xyz="0.345 0.0 -0.0235" rpy="0.0 0.0 0.0"/>
-    <axis xyz="0.0 0.0 1.0"/>
-    <limit lower="${-pi}" upper="${pi}" effort="10.0" velocity="${10*pi}"/>
-  </joint> -->
 </robot>

Commit message: add depart link

File: src/kirin/urdf/kirin.urdf.xacro (robot description, xacro)
@@ -41,4 +41,5 @@
   </link>
   <link name="phi_link"/>
+  <link name="depart"/>
   <!-- joint settings -->
   <joint name="theta_joint" type="continuous">
@@ -69,3 +70,8 @@
     <limit lower="${-pi}" upper="${pi}" effort="10.0" velocity="${10*pi}"/>
   </joint>
+  <joint name="depart_joint" type="fixed">
+    <parent link="fix_base"/>
+    <child link="depart"/>
+    <origin xyz="0.55 0.55 0.225" rpy="0.0 0.0 ${-pi/2}"/>
+  </joint>
 </robot>

Commit message: change depart position

File: src/kirin/urdf/kirin.urdf.xacro (robot description, xacro)
@@ -73,5 +73,5 @@
     <parent link="fix_base"/>
     <child link="depart"/>
-    <origin xyz="0.55 0.55 0.225" rpy="0.0 0.0 ${-pi/2}"/>
+    <origin xyz="0.65 0.55 0.225" rpy="0.0 0.0 ${-pi/2}"/>
   </joint>
 </robot>

Commit message: urdf file adapt to field change

File: src/kirin/urdf/kirin.urdf.xacro (robot description, xacro)
@@ -1,3 +1,5 @@
 <robot name="kirin" xmlns:xacro="http://ros.org/wiki/xacro">
+  <xacro:arg name="field" default="red" />
+  <xacro:property name="field" default="$(arg field)" />
   <material name="default">
     <color rgba="0.7 0.7 0.7 1.0"/>
@@ -73,5 +75,10 @@
     <parent link="fix_base"/>
     <child link="depart"/>
-    <origin xyz="0.65 0.55 0.225" rpy="0.0 0.0 ${-pi/2}"/>
+    <xacro:if value="${field=='red'}">
+      <origin xyz="0.65 0.55 0.225" rpy="0.0 0.0 ${-pi/2}"/>
+    </xacro:if>
+    <xacro:if value="${field=='blue'}">
+      <origin xyz="0.65 -0.55 0.225" rpy="0.0 0.0 ${pi/2}"/>
+    </xacro:if>
   </joint>
 </robot>

Commit message: add initial depart and share wait frame

File: src/kirin/urdf/kirin.urdf.xacro (robot description, xacro)
@@ -44,4 +44,5 @@
   <link name="phi_link"/>
   <link name="depart"/>
+  <link name="initial_depart"/>
   <!-- joint settings -->
   <joint name="theta_joint" type="continuous">
@@ -82,3 +83,13 @@
     </xacro:if>
   </joint>
+  <joint name="initial_depart_joint" type="fixed">
+    <parent link="fix_base"/>
+    <child link="initial_depart"/>
+    <xacro:if value="${field=='red'}">
+      <origin xyz="0.65 -0.7 0.225" rpy="0.0 0.0 0.0"/>
+    </xacro:if>
+    <xacro:if value="${field=='blue'}">
+      <origin xyz="0.65 0.7 0.225" rpy="0.0 0.0 0.0"/>
+    </xacro:if>
+  </joint>
 </robot>

Commit message: change home command, fix parameter and modify depart point

File: src/kirin/urdf/kirin.urdf.xacro (robot description, xacro)
@@ -77,8 +77,8 @@
     <child link="depart"/>
     <xacro:if value="${field=='red'}">
-      <origin xyz="0.65 0.55 0.225" rpy="0.0 0.0 ${-pi/2}"/>
+      <origin xyz="0.60 0.55 0.225" rpy="0.0 0.0 ${-pi/2}"/>
     </xacro:if>
     <xacro:if value="${field=='blue'}">
-      <origin xyz="0.65 -0.55 0.225" rpy="0.0 0.0 ${pi/2}"/>
+      <origin xyz="0.60 -0.55 0.225" rpy="0.0 0.0 ${pi/2}"/>
     </xacro:if>
   </joint>
@@ -87,8 +87,8 @@
     <child link="initial_depart"/>
     <xacro:if value="${field=='red'}">
-      <origin xyz="0.65 -0.7 0.225" rpy="0.0 0.0 0.0"/>
+      <origin xyz="0.60 -0.65 0.225" rpy="0.0 0.0 0.0"/>
     </xacro:if>
     <xacro:if value="${field=='blue'}">
-      <origin xyz="0.65 0.7 0.225" rpy="0.0 0.0 0.0"/>
+      <origin xyz="0.60 0.65 0.225" rpy="0.0 0.0 0.0"/>
     </xacro:if>
   </joint>

Commit message: modify initial automation

File: src/kirin/urdf/kirin.urdf.xacro (robot description, xacro)
@@ -87,8 +87,8 @@
     <child link="initial_depart"/>
     <xacro:if value="${field=='red'}">
-      <origin xyz="0.60 -0.65 0.225" rpy="0.0 0.0 0.0"/>
+      <origin xyz="0.60 -0.60 0.225" rpy="0.0 0.0 0.0"/>
     </xacro:if>
     <xacro:if value="${field=='blue'}">
-      <origin xyz="0.60 0.65 0.225" rpy="0.0 0.0 0.0"/>
+      <origin xyz="0.60 0.60 0.225" rpy="0.0 0.0 0.0"/>
     </xacro:if>
   </joint>
